Commit message: v0.2

File: urdf/x_shape.urdf (robot description, URDF)
Before this commit: robot x_shape, 2 links, 1 joints
Links:
- added link part0, mass 80; collision box size=0.98 0.92 0.41; visual box size=0.98 0.92 0.41
- link part1: mass 1.0 -> 10
- link part2: mass 1.0 -> 10
Joints:
- removed joint x_joint
- added joint x_joint1: type fixed, parent part0, child part1, origin xyz=0 0 -.22
- added joint x_joint2: type fixed, parent part0, child part2, origin xyz=0 0 -.22
