Commit message: multi-angle and base size
simulation of multiple angles and base sizes

File: urdf/drone.urdf (robot description, URDF)
Before this commit: robot x_shape, 3 links, 2 joints
Links:
- removed link part0
- removed link part1
- removed link part2
- added link link1, mass 80; collision box size=0.98 0.92 0.41; visual box size=0.98 0.92 0.41
- added link link2, mass 10; collision box size=8 0.05 0.05; visual box size=8 0.05 0.05
- added link link3, mass 10; collision box size=8 0.05 0.05; visual box size=8 0.05 0.05
Joints:
- joint x_joint1: child part1 -> link2; origin xyz=0 0 -.22 -> xyz=0 0 -.20; parent part0 -> link1
- joint x_joint2: child part2 -> link3; origin xyz=0 0 -.22 -> xyz=0 0 -.20; parent part0 -> link1

Commit message: add plot

File: urdf/drone.urdf (robot description, URDF)
Before this commit: robot x_shape, 3 links, 2 joints
Links:
- link link1: geometry collision box size=1 1 0.4; visual box size=1 1 0.4
